File: battery-tester/battery-tester.kicad_sch (KiCad schematic)
At the start: 0 parts

Commit message: final
Parts:
- added C1: 100nF, Capacitor_THT:C_Disc_D5.0mm_W2.5mm_P5.00mm, symbol Device:C
- added D1: RED, LED_THT:LED_D5.0mm, symbol Device:LED
- added D2: YELLOW, LED_THT:LED_D5.0mm, symbol Device:LED
- added D3: GREEN, LED_THT:LED_D5.0mm, symbol Device:LED
- added D4, D5: 1N4148, Diode_THT:D_DO-35_SOD27_P7.62mm_Horizontal, symbol Diode:1N4148
- added J1: Battery, TerminalBlock_Phoenix:TerminalBlock_Phoenix_MKDS-1,5-2_1x02_P5.00mm_Horizontal, symbol Connector:Screw_Terminal_01x02
- added R1: 22k, Resistor_THT:R_Axial_DIN0207_L6.3mm_D2.5mm_P7.62mm_Horizontal, symbol Device:R
- added R2, R4: 10k, Resistor_THT:R_Axial_DIN0207_L6.3mm_D2.5mm_P7.62mm_Horizontal, symbol Device:R
- added R3: 18k, Resistor_THT:R_Axial_DIN0207_L6.3mm_D2.5mm_P7.62mm_Horizontal, symbol Device:R
- added R5, R6, R7, R8: 2.2k, Resistor_THT:R_Axial_DIN0207_L6.3mm_D2.5mm_P7.62mm_Horizontal, symbol Device:R
- added U1: LM393, Package_DIP:DIP-8_W7.62mm, symbol Comparator:LM393
- added U2: TL431LP, Package_TO_SOT_THT:TO-92_Inline, symbol Reference_Voltage:TL431LP
Connections:
- new net: D1.1 (K), D5.1 (K), U1.7
- new net: D1.2 (A), R8.2
- new net: D2.2 (A), D4.2 (A), D5.2 (A), R7.2
- new net: R3.2, R4.1, U1.5 (+)
- new net: R5.2, U1.3 (+), U1.6 (-), U2.1 (REF), U2.3 (K)
- new net: R1.2, R2.1, U1.2 (-)
- new net: D3.1 (K), D4.1 (K), U1.1
- new net: D3.2 (A), R6.2
- new net +BATT: C1.1, J1.1 (Pin_1), R1.1, R3.1, R5.1, R6.1, R7.1, R8.1, U1.8 (V+)
- new net GND: C1.2, D2.1 (K), J1.2 (Pin_2), R2.2, R4.2, U1.4 (V-), U2.2 (A)
